Commit message: config

File: launch/include/config/robot.urdf.xacro (robot description, xacro)
@@ -19,5 +19,5 @@
     <parent link="chassis_link" />
     <child link="velodyne" />
-    <origin xyz="0 0 0" rpy="0 0 0" />
+    <origin xyz="1.33 0 1.33" rpy="0 0 0" />
   </joint>
   <link name="navsat_link"> </link>
